Commit message: braxionas_edit

File: braxionas/src/braxionas/urdf/braxionas.xacro (robot description, xacro)
@@ -26,4 +26,10 @@
             <material name="${xrvma}" />
         </visual>
+        <collision>
+            <geometry>
+               <mesh filename ="package://braxionas/meshes/${fakelos}/${onoma}" scale="0.001 0.001 0.001" />
+            </geometry>
+            <origin xyz="${x} ${y} ${z}" rpy="${rpyx} ${rpyy} 0"/>
+        </collision>
        </link>
     </xacro:macro>
