Commit message: lidar_edit2

File: my_robot_description/src/my_robot_description/urdf/lidar.xacro (robot description, xacro)
@@ -2,5 +2,5 @@
 <robot xmlns:xacro="http://www.ros.org/wiki/xacro">
     <xacro:property name="lidar_length" value="0.05"/>
-    <xacro:property name="lidar_radius" value="0.1"/>
+    <xacro:property name="lidar_radius" value="0.05"/>
     <link name="lidar_link">
             <visual>
@@ -27,13 +27,13 @@
     <gazebo reference="lidar_link">
         <material>Gazebo/Red</material>
-        <self_collide>true</self_collide>
+        <self_collide>false</self_collide>
         <sensor type="ray" name="head_hokuyo_sensor">
-             <pose>0 0 0 0 0 0</pose>
+             <pose>10 0 10 0 0 0</pose>
              <visualize>true</visualize>
-             <update_rate>40</update_rate>
+             <update_rate>30</update_rate>
             <ray>
              <scan>
               <horizontal>
-                <samples>360</samples>
+                <samples>720</samples>
                 <resolution>1</resolution>
                 <min_angle>-0.0872665</min_angle>
@@ -53,6 +53,7 @@
             </ray>
             <plugin name="gazebo_ros_ray_sensor" filename="libgazebo_ros_ray_sensor.so">
-                <topicName>/scan</topicName>
-                <frameName>lidar_link</frameName>
+                   <topic_name>/scan</topic_name>
+                   <frame_name>lidar_link</frame_name>
+                   <output_type>sensor_msgs/LaserScan</output_type>
             </plugin>
         </sensor>
