Commit message: Gazebo_qr_object_edit

File: my_robot_description/src/my_robot_description/urdf/mobile_base.xacro (robot description, xacro)
@@ -6,5 +6,4 @@
     <xacro:property name="wheel_radius" value="0.1" />
     <xacro:property name="wheel_length" value="0.05" />
-    <link name="base_footprint" />
     <link name="base_link">
         <visual>

File: my_robot_description/src/my_robot_description/urdf/my_robot.urdf.xacro (robot description, xacro)
@@ -1,4 +1,5 @@
 <?xml version="1.0"?>
 <robot name="my_robot" xmlns:xacro="http://www.ros.org/wiki/xacro">
+   <link name="base_footprint" />
     <xacro:include filename="common_properties.xacro" />
     <xacro:include filename="mobile_base.xacro" />
@@ -7,3 +8,4 @@
     <xacro:include filename="lidar.xacro" />
     <xacro:include filename="lidar2.xacro" />
+    <!--<xacro:include filename="ur5.xacro" />-->
 </robot>
