Commit message: edit_marker_rviz

File: my_robot_description/src/my_robot_description/urdf/lidar2.xacro (robot description, xacro)
@@ -23,5 +23,5 @@
          <parent link="lidar_link"/>
          <child link="lidar_link2" />
-         <origin xyz="0 0 ${lidar_length2 + 0.01}" rpy="0 0 ${pi / 2.0} " />
+         <origin xyz="0 0 ${lidar_length2 + 0.01}" rpy="0 0 0 " />
      </joint>
     <gazebo reference="lidar_link2">

Commit message: ransac_edit

File: my_robot_description/src/my_robot_description/urdf/lidar2.xacro (robot description, xacro)
@@ -23,5 +23,5 @@
          <parent link="lidar_link"/>
          <child link="lidar_link2" />
-         <origin xyz="0 0 ${lidar_length2 + 0.01}" rpy="0 0 0 " />
+         <origin xyz="0 0 ${lidar_length2 + 0.01}" rpy="0 0 ${-pi / 2.0} " />
      </joint>
     <gazebo reference="lidar_link2">

File: my_robot_description/src/my_robot_description/urdf/my_robot.urdf.xacro (robot description, xacro)
@@ -6,6 +6,7 @@
     <xacro:include filename="mobile_base_gazebo.xacro" />
     <xacro:include filename="camera.xacro" />
+    <xacro:include filename="camera2.xacro" />
     <xacro:include filename="lidar.xacro" />
     <xacro:include filename="lidar2.xacro" />
-    <!--<xacro:include filename="ur5.xacro" />-->
+    <!--xacro:include filename="ur5.xacro"  -->
 </robot>

File: my_robot_description/src/my_robot_description/urdf/ur5.xacro (robot description, xacro)
@@ -321,5 +321,5 @@
     <plugin name="gazebo_ros_joint_state_publisher"
         filename="libgazebo_ros_joint_state_publisher.so">
-       <update_rate>10</update_rate>
+       <update_rate>50</update_rate>
        <joint_name>shoulder_pan_joint</joint_name>
        <joint_name>shoulder_lift_joint</joint_name>
@@ -334,5 +334,5 @@
                 filename="libgazebo_ros_joint_pose_trajectory.so">
             <!-- Update rate in Hz -->
-            <update_rate>2</update_rate>
+            <update_rate>50</update_rate>
         </plugin>
     </gazebo>
