Commit message: edit_ur5_gazebo

File: my_robot_description/src/my_robot_description/urdf/my_robot.urdf.xacro (robot description, xacro)
@@ -10,4 +10,4 @@
     <!--<xacro:include filename="arm_gazebo.xacro" />
     <xacro:include filename="arm.xacro" />  -->
-    <!--<xacro:include filename="ur5.xacro" />-->
+    <xacro:include filename="ur5.xacro" />
 </robot>

File: my_robot_description/src/my_robot_description/urdf/ur5.xacro (robot description, xacro)
@@ -28,6 +28,6 @@
    <xacro:property name="upper_arm_pitch" value="0" />
    <xacro:property name="upper_arm_yaw" value="0" />
-   <xacro:property name="shoulder_lift_lower_limit" value="-6.2832" />
-   <xacro:property name="shoulder_lift_upper_limit" value="6.2832" />
+   <xacro:property name="shoulder_lift_lower_limit" value="${-pi/2}" />
+   <xacro:property name="shoulder_lift_upper_limit" value="0" />
    <xacro:property name="shoulder_lift_velocity_limit" value="3.1416" />
    <xacro:property name="shoulder_lift_effort_limit" value="150.0" />
@@ -100,68 +100,9 @@
     </inertial>
   </xacro:macro>
-    <xacro:macro name="ur5_transmission" params="prefix">
-    <transmission name="${prefix}shoulder_pan_trans">
-      <type>transmission_interface/SimpleTransmission</type>
-      <joint name="${prefix}shoulder_pan_joint">
-        <hardwareInterface>hardware_interface/PositionJointInterface</hardwareInterface>
-      </joint>
-      <actuator name="${prefix}shoulder_pan_motor">
-        <mechanicalReduction>1</mechanicalReduction>
-      </actuator>
-    </transmission>
-    <transmission name="${prefix}shoulder_lift_trans">
-      <type>transmission_interface/SimpleTransmission</type>
-      <joint name="${prefix}shoulder_lift_joint">
-        <hardwareInterface>hardware_interface/PositionJointInterface</hardwareInterface>
-      </joint>
-      <actuator name="${prefix}shoulder_lift_motor">
-        <mechanicalReduction>1</mechanicalReduction>
-      </actuator>
-    </transmission>
-    <transmission name="${prefix}elbow_trans">
-      <type>transmission_interface/SimpleTransmission</type>
-      <joint name="${prefix}elbow_joint">
-        <hardwareInterface>hardware_interface/PositionJointInterface</hardwareInterface>
-      </joint>
-      <actuator name="${prefix}elbow_motor">
-        <mechanicalReduction>1</mechanicalReduction>
-      </actuator>
-    </transmission>
-    <transmission name="${prefix}wrist_1_trans">
-      <type>transmission_interface/SimpleTransmission</type>
-      <joint name="${prefix}wrist_1_joint">
-        <hardwareInterface>hardware_interface/PositionJointInterface</hardwareInterface>
-      </joint>
-      <actuator name="${prefix}wrist_1_motor">
-        <mechanicalReduction>1</mechanicalReduction>
-      </actuator>
-    </transmission>
-    <transmission name="${prefix}wrist_2_trans">
-      <type>transmission_interface/SimpleTransmission</type>
-      <joint name="${prefix}wrist_2_joint">
-        <hardwareInterface>hardware_interface/PositionJointInterface</hardwareInterface>
-      </joint>
-      <actuator name="${prefix}wrist_2_motor">
-        <mechanicalReduction>1</mechanicalReduction>
-      </actuator>
-    </transmission>
-    <transmission name="${prefix}wrist_3_trans">
-      <type>transmission_interface/SimpleTransmission</type>
-      <joint name="${prefix}wrist_3_joint">
-        <hardwareInterface>hardware_interface/PositionJointInterface</hardwareInterface>
-      </joint>
-      <actuator name="${prefix}wrist_3_motor">
-        <mechanicalReduction>1</mechanicalReduction>
-      </actuator>
-    </transmission>
-  </xacro:macro>
-  <xacro:ur5_transmission
-      prefix=""
-    />
  <link name="base_ur5" >
     <visual>
         <origin xyz="0 0 0" rpy="0 0 ${pi}"/>
         <geometry>
-          <mesh filename="package://my_robot_description/meshes/visual/base.dae" />
+         <mesh filename="file:///home/hercules/my_robot_description/install/my_robot_description/share/my_robot_description/meshes/visual/base.dae"/>
         </geometry>
         <material name="LightGrey">
@@ -172,5 +113,5 @@
         <origin xyz="0 0 0" rpy="0 0 ${pi}"/>
         <geometry>
-          <mesh filename="package://my_robot_description/meshes/collision/base.stl" />
+          <mesh filename="file:///home/hercules/my_robot_description/install/my_robot_description/share/my_robot_description/meshes/collision/base.stl"/>
         </geometry>
     </collision>
@@ -183,5 +124,5 @@
         <origin xyz="0 0 0" rpy="0 0 ${pi}"/>
         <geometry>
-          <mesh filename="package://my_robot_description/meshes/visual/shoulder.dae"/>
+          <mesh filename="file:///home/hercules/my_robot_description/install/my_robot_description/share/my_robot_description/meshes/visual/shoulder.dae"/>
         </geometry>
         <material name="LightGrey">
@@ -192,5 +133,5 @@
         <origin xyz="0 0 0" rpy="0 0 ${pi}"/>
         <geometry>
-          <mesh filename="package://my_robot_description/meshes/collision/shoulder.stl"/>
+          <mesh filename="file:///home/hercules/my_robot_description/install/my_robot_description/share/my_robot_description/meshes/collision/shoulder.stl"/>
         </geometry>
       </collision>
@@ -203,5 +144,5 @@
         <origin xyz="0 0 ${shoulder_offset}" rpy="${pi/2} 0 ${-pi/2}"/>
         <geometry>
-          <mesh filename="package://my_robot_description/meshes/visual/upperarm.dae"/>
+          <mesh filename="file:///home/hercules/my_robot_description/install/my_robot_description/share/my_robot_description/meshes/visual/upperarm.dae"/>
         </geometry>
         <material name="LightGrey">
@@ -212,5 +153,5 @@
         <origin xyz="0 0 ${shoulder_offset}" rpy="${pi/2} 0 ${-pi/2}"/>
         <geometry>
-          <mesh filename="package://my_robot_description/meshes/collision/upperarm.stl"/>
+          <mesh filename="file:///home/hercules/my_robot_description/install/my_robot_description/share/my_robot_description/meshes/collision/upperarm.stl"/>
         </geometry>
       </collision>
@@ -223,5 +164,5 @@
         <origin xyz="0 0 ${elbow_offset}" rpy="${pi/2} 0 ${-pi/2}"/>
         <geometry>
-          <mesh filename="package://my_robot_description/meshes/visual/forearm.dae"/>
+          <mesh filename="file:///home/hercules/my_robot_description/install/my_robot_description/share/my_robot_description/meshes/visual/forearm.dae"/>
         </geometry>
         <material name="LightGrey">
@@ -232,5 +173,5 @@
         <origin xyz="0 0 ${elbow_offset}" rpy="${pi/2} 0 ${-pi/2}"/>
         <geometry>
-          <mesh filename="package://my_robot_description/meshes/collision/forearm.stl"/>
+          <mesh filename="file:///home/hercules/my_robot_description/install/my_robot_description/share/my_robot_description/meshes/collision/forearm.stl"/>
         </geometry>
       </collision>
@@ -243,5 +184,5 @@
         <origin xyz="0 0 ${wrist_1_visual_offset}" rpy="${pi/2} 0 0"/>
         <geometry>
-          <mesh filename="package://my_robot_description/meshes/visual/wrist1.dae"/>
+          <mesh filename="file:///home/hercules/my_robot_description/install/my_robot_description/share/my_robot_description/meshes/visual/wrist1.dae"/>
         </geometry>
         <material name="LightGrey">
@@ -252,5 +193,5 @@
         <origin xyz="0 0 ${wrist_1_visual_offset}" rpy="${pi/2} 0 0"/>
         <geometry>
-          <mesh filename="package://my_robot_description/meshes/collision/wrist1.stl"/>
+          <mesh filename="file:///home/hercules/my_robot_description/install/my_robot_description/share/my_robot_description/meshes/collision/wrist1.stl"/>
         </geometry>
       </collision>
@@ -263,5 +204,5 @@
         <origin xyz="0 0 ${wrist_2_visual_offset}" rpy="0 0 0"/>
         <geometry>
-          <mesh filename="package://my_robot_description/meshes/visual/wrist2.dae"/>
+          <mesh filename="file:///home/hercules/my_robot_description/install/my_robot_description/share/my_robot_description/meshes/visual/wrist2.dae"/>
         </geometry>
         <material name="LightGrey">
@@ -272,5 +213,5 @@
         <origin xyz="0 0 ${wrist_2_visual_offset}" rpy="0 0 0"/>
         <geometry>
-          <mesh filename="package://my_robot_description/meshes/collision/wrist2.stl"/>
+          <mesh filename="file:///home/hercules/my_robot_description/install/my_robot_description/share/my_robot_description/meshes/collision/wrist2.stl"/>
         </geometry>
       </collision>
@@ -283,5 +224,5 @@
         <origin xyz="0 0 ${wrist_3_visual_offset}" rpy="${pi/2} 0 0"/>
         <geometry>
-          <mesh filename="package://my_robot_description/meshes/visual/wrist3.dae"/>
+          <mesh filename="file:///home/hercules/my_robot_description/install/my_robot_description/share/my_robot_description/meshes/visual/wrist3.dae"/>
         </geometry>
         <material name="LightGrey">
@@ -292,5 +233,5 @@
         <origin xyz="0 0 ${wrist_3_visual_offset}" rpy="${pi/2} 0 0"/>
         <geometry>
-          <mesh filename="package://my_robot_description/meshes/collision/wrist3.stl"/>
+          <mesh filename="file:///home/hercules/my_robot_description/install/my_robot_description/share/my_robot_description/meshes/collision/wrist3.stl"/>
         </geometry>
       </collision>
@@ -303,5 +244,5 @@
         <parent link="lidar_link2" />
         <child link ="base_ur5" />
-        <origin xyz ="0 0 ${lidar_length2 }" rpy="0 0 ${pi}" />
+        <origin xyz ="0 0 ${lidar_length2 }" rpy="0 0 ${-pi}" />
     </joint>
     <joint name="shoulder_pan_joint" type="revolute">
@@ -377,10 +318,8 @@
       <dynamics damping="1.0" friction="1.0"/>
     </joint>
-    <gazebo>
+   <gazebo>
     <plugin name="gazebo_ros_joint_state_publisher"
         filename="libgazebo_ros_joint_state_publisher.so">
-      <!-- Update rate in Hertz -->
        <update_rate>10</update_rate>
-      <!-- Name of joints in the model whose states will be published. -->
        <joint_name>shoulder_pan_joint</joint_name>
        <joint_name>shoulder_lift_joint</joint_name>
@@ -391,3 +330,10 @@
     </plugin>
   </gazebo>
+  <gazebo>
+        <plugin name="joint_pose_trajectory_controller"
+                filename="libgazebo_ros_joint_pose_trajectory.so">
+            <!-- Update rate in Hz -->
+            <update_rate>2</update_rate>
+        </plugin>
+    </gazebo>
 </robot>

Commit message: moveit2

File: my_robot_description/src/my_robot_description/urdf/my_robot.urdf.xacro (robot description, xacro)
@@ -9,4 +9,4 @@
     <xacro:include filename="lidar.xacro" />
     <xacro:include filename="lidar2.xacro" />
-    <!--xacro:include filename="ur5.xacro"  -->
+    <xacro:include filename="ur5.xacro" />
 </robot>

File: my_robot_description/src/my_robot_description/urdf/ur5.xacro (robot description, xacro)
@@ -244,5 +244,5 @@
         <parent link="lidar_link2" />
         <child link ="base_ur5" />
-        <origin xyz ="0 0 ${lidar_length2 }" rpy="0 0 ${-pi}" />
+        <origin xyz ="0 0 ${lidar_length2}" rpy="0 0 ${-pi}" />
     </joint>
     <joint name="shoulder_pan_joint" type="revolute">
