Commit message: lidar_edit

File: my_robot_description/src/my_robot_description/urdf/camera.xacro (robot description, xacro)
@@ -22,5 +22,5 @@
          <parent link="base_link"/>
          <child link="camera_link" />
-         <origin xyz="0 ${(base_width / 2.0)+0.01} ${(base_height / 2.0)+ 0.05}" rpy="0 0 ${pi/2}" />
+         <origin xyz="0 ${(base_width / 2.0)} ${(base_height / 2.0)+ 0.05}" rpy="0 0 ${pi/2}" />
      </joint>
      <link name="camera_link_optical">

File: my_robot_description/src/my_robot_description/urdf/common_properties.xacro (robot description, xacro)
@@ -6,4 +6,7 @@
     <material name="grey">
         <color rgba="0.5 0.5 0.5 1" />
+    </material>
+        <material name="red">
+        <color rgba="0.5 0 0 1" />
     </material>
     <xacro:macro name="box_inertia" params="m l w h xyz rpy">

File: my_robot_description/src/my_robot_description/urdf/my_robot.urdf.xacro (robot description, xacro)
@@ -5,3 +5,4 @@
     <xacro:include filename="mobile_base_gazebo.xacro" />
     <xacro:include filename="camera.xacro" />
+    <xacro:include filename="lidar.xacro" />
 </robot>

Commit message: edit_marker

File: my_robot_description/src/my_robot_description/urdf/camera.xacro (robot description, xacro)
@@ -24,4 +24,9 @@
          <origin xyz="0 ${(base_width / 2.0)} ${(base_height / 2.0)+ 0.05}" rpy="0 0 ${pi/2}" />
      </joint>
+     <!--<joint name="base_camera_joint" type="fixed">
+         <parent link="hand_link"/>
+         <child link="camera_link" />
+         <origin xyz="0.02 0 0.3" rpy="0 0 0" />
+     </joint>-->
      <link name="camera_link_optical">
      </link>

File: my_robot_description/src/my_robot_description/urdf/my_robot.urdf.xacro (robot description, xacro)
@@ -8,4 +8,6 @@
     <xacro:include filename="lidar.xacro" />
     <xacro:include filename="lidar2.xacro" />
+    <!--<xacro:include filename="arm_gazebo.xacro" />
+    <xacro:include filename="arm.xacro" />  -->
     <!--<xacro:include filename="ur5.xacro" />-->
 </robot>

File: my_robot_description/src/my_robot_description/urdf/ur5.xacro (robot description, xacro)
@@ -88,4 +88,7 @@
     <xacro:property name="wrist_3_velocity_limit" value="3.1416" />
     <xacro:property name="wrist_3_effort_limit" value="28.0" />
+    <xacro:property name="safety_limits" default="false"/>
+    <xacro:property name="safety_pos_margin" default="0.15"/>
+    <xacro:property name="safety_k_position" default="20"/>
   <xacro:macro name="cylinder_inertial2" params="radius length mass *origin">
     <inertial>
@@ -97,4 +100,63 @@
     </inertial>
   </xacro:macro>
+    <xacro:macro name="ur5_transmission" params="prefix">
+    <transmission name="${prefix}shoulder_pan_trans">
+      <type>transmission_interface/SimpleTransmission</type>
+      <joint name="${prefix}shoulder_pan_joint">
+        <hardwareInterface>hardware_interface/PositionJointInterface</hardwareInterface>
+      </joint>
+      <actuator name="${prefix}shoulder_pan_motor">
+        <mechanicalReduction>1</mechanicalReduction>
+      </actuator>
+    </transmission>
+    <transmission name="${prefix}shoulder_lift_trans">
+      <type>transmission_interface/SimpleTransmission</type>
+      <joint name="${prefix}shoulder_lift_joint">
+        <hardwareInterface>hardware_interface/PositionJointInterface</hardwareInterface>
+      </joint>
+      <actuator name="${prefix}shoulder_lift_motor">
+        <mechanicalReduction>1</mechanicalReduction>
+      </actuator>
+    </transmission>
+    <transmission name="${prefix}elbow_trans">
+      <type>transmission_interface/SimpleTransmission</type>
+      <joint name="${prefix}elbow_joint">
+        <hardwareInterface>hardware_interface/PositionJointInterface</hardwareInterface>
+      </joint>
+      <actuator name="${prefix}elbow_motor">
+        <mechanicalReduction>1</mechanicalReduction>
+      </actuator>
+    </transmission>
+    <transmission name="${prefix}wrist_1_trans">
+      <type>transmission_interface/SimpleTransmission</type>
+      <joint name="${prefix}wrist_1_joint">
+        <hardwareInterface>hardware_interface/PositionJointInterface</hardwareInterface>
+      </joint>
+      <actuator name="${prefix}wrist_1_motor">
+        <mechanicalReduction>1</mechanicalReduction>
+      </actuator>
+    </transmission>
+    <transmission name="${prefix}wrist_2_trans">
+      <type>transmission_interface/SimpleTransmission</type>
+      <joint name="${prefix}wrist_2_joint">
+        <hardwareInterface>hardware_interface/PositionJointInterface</hardwareInterface>
+      </joint>
+      <actuator name="${prefix}wrist_2_motor">
+        <mechanicalReduction>1</mechanicalReduction>
+      </actuator>
+    </transmission>
+    <transmission name="${prefix}wrist_3_trans">
+      <type>transmission_interface/SimpleTransmission</type>
+      <joint name="${prefix}wrist_3_joint">
+        <hardwareInterface>hardware_interface/PositionJointInterface</hardwareInterface>
+      </joint>
+      <actuator name="${prefix}wrist_3_motor">
+        <mechanicalReduction>1</mechanicalReduction>
+      </actuator>
+    </transmission>
+  </xacro:macro>
+  <xacro:ur5_transmission
+      prefix=""
+    />
  <link name="base_ur5" >
     <visual>
@@ -250,4 +312,7 @@
       <limit lower="${shoulder_pan_lower_limit}" upper="${shoulder_pan_upper_limit}"
         effort="${shoulder_pan_effort_limit}" velocity="${shoulder_pan_velocity_limit}"/>
+      <xacro:if value="${safety_limits}">
+         <safety_controller soft_lower_limit="${shoulder_pan_lower_limit + safety_pos_margin}" soft_upper_limit="${shoulder_pan_upper_limit - safety_pos_margin}" k_position="${safety_k_position}" k_velocity="0.0"/>
+      </xacro:if>
       <dynamics damping="50.0" friction="1.0"/>
     </joint>
@@ -259,4 +324,7 @@
       <limit lower="${shoulder_lift_lower_limit}" upper="${shoulder_lift_upper_limit}"
         effort="${shoulder_lift_effort_limit}" velocity="${shoulder_lift_velocity_limit}"/>
+      <xacro:if value="${safety_limits}">
+         <safety_controller soft_lower_limit="${shoulder_lift_lower_limit + safety_pos_margin}" soft_upper_limit="${shoulder_lift_upper_limit - safety_pos_margin}" k_position="${safety_k_position}" k_velocity="0.0"/>
+      </xacro:if>
       <dynamics damping="50.0" friction="1.0"/>
     </joint>
@@ -268,4 +336,7 @@
       <limit lower="${elbow_joint_lower_limit}" upper="${elbow_joint_upper_limit}"
         effort="${elbow_joint_effort_limit}" velocity="${elbow_joint_velocity_limit}"/>
+      <xacro:if value="${safety_limits}">
+         <safety_controller soft_lower_limit="${elbow_joint_lower_limit + safety_pos_margin}" soft_upper_limit="${elbow_joint_upper_limit - safety_pos_margin}" k_position="${safety_k_position}" k_velocity="0.0"/>
+      </xacro:if>
       <dynamics damping="10.0" friction="1.0"/>
     </joint>
@@ -277,4 +348,7 @@
       <limit lower="${wrist_1_lower_limit}" upper="${wrist_1_upper_limit}"
         effort="${wrist_1_effort_limit}" velocity="${wrist_1_velocity_limit}"/>
+      <xacro:if value="${safety_limits}">
+         <safety_controller soft_lower_limit="${wrist_1_lower_limit + safety_pos_margin}" soft_upper_limit="${wrist_1_upper_limit - safety_pos_margin}" k_position="${safety_k_position}" k_velocity="0.0"/>
+      </xacro:if>
       <dynamics damping="5.0" friction="1.0"/>
     </joint>
@@ -286,4 +360,7 @@
       <limit lower="${wrist_2_lower_limit}" upper="${wrist_2_upper_limit}"
              effort="${wrist_2_effort_limit}" velocity="${wrist_2_velocity_limit}"/>
+      <xacro:if value="${safety_limits}">
+         <safety_controller soft_lower_limit="${wrist_2_lower_limit + safety_pos_margin}" soft_upper_limit="${wrist_2_upper_limit - safety_pos_margin}" k_position="${safety_k_position}" k_velocity="0.0"/>
+      </xacro:if>
       <dynamics damping="2.0" friction="1.0"/>
     </joint>
@@ -295,5 +372,22 @@
       <limit lower="${wrist_3_lower_limit}" upper="${wrist_3_upper_limit}"
              effort="${wrist_3_effort_limit}" velocity="${wrist_3_velocity_limit}"/>
+      <xacro:if value="${safety_limits}">
+         <safety_controller soft_lower_limit="${wrist_3_lower_limit + safety_pos_margin}" soft_upper_limit="${wrist_3_upper_limit - safety_pos_margin}" k_position="${safety_k_position}" k_velocity="0.0"/>
+      </xacro:if>
       <dynamics damping="1.0" friction="1.0"/>
     </joint>
+    <gazebo>
+    <plugin name="gazebo_ros_joint_state_publisher"
+        filename="libgazebo_ros_joint_state_publisher.so">
+      <!-- Update rate in Hertz -->
+       <update_rate>10</update_rate>
+      <!-- Name of joints in the model whose states will be published. -->
+       <joint_name>shoulder_pan_joint</joint_name>
+       <joint_name>shoulder_lift_joint</joint_name>
+       <joint_name>elbow_joint</joint_name>
+       <joint_name>wrist_1_joint</joint_name>
+       <joint_name>wrist_2_joint</joint_name>
+       <joint_name>wrist_3_joint</joint_name>
+    </plugin>
+  </gazebo>
 </robot>

Commit message: camera_edit

File: my_robot_description/src/my_robot_description/urdf/camera.xacro (robot description, xacro)
@@ -40,4 +40,24 @@
     </joint>
      <gazebo reference="camera_link">
+     <material>Gazebo/ZincYellow</material>
+     <sensor name="camera_sensor" type="camera">
+     <pose>0 0 0 0 0 0</pose>
+     <visualize>true</visualize>
+     <update_rate>10.0</update_rate>
+      <camera>
+       <horizontal_fov>1.3962634</horizontal_fov>
+       <image>
+         <width>1280</width>
+         <height>720</height>
+         <format>R8G8B8</format>
+       </image>
+      </camera>
+     <plugin name="camera_controller" filename="libgazebo_ros_camera.so">
+      <frame_name>camera_link_optical</frame_name>
+     </plugin>
+     </sensor>
+    </gazebo>
+ <!--
+     <gazebo reference="camera_link">
         <material>Gazebo/ZincYellow</material>
         <sensor name="camera_sensor" type="camera">
@@ -49,4 +69,4 @@
             </plugin>
         </sensor>
-     </gazebo>
+     </gazebo>-->
 </robot>

File: my_robot_description/src/my_robot_description/urdf/my_robot.urdf.xacro (robot description, xacro)
@@ -8,6 +8,4 @@
     <xacro:include filename="lidar.xacro" />
     <xacro:include filename="lidar2.xacro" />
-    <!--<xacro:include filename="arm_gazebo.xacro" />
-    <xacro:include filename="arm.xacro" />  -->
-    <xacro:include filename="ur5.xacro" />
+    <!--<xacro:include filename="ur5.xacro" />-->
 </robot>

File: my_robot_description/src/my_robot_description/urdf/ur5.xacro (robot description, xacro)
@@ -28,6 +28,6 @@
    <xacro:property name="upper_arm_pitch" value="0" />
    <xacro:property name="upper_arm_yaw" value="0" />
-   <xacro:property name="shoulder_lift_lower_limit" value="${-pi/2}" />
-   <xacro:property name="shoulder_lift_upper_limit" value="0" />
+   <xacro:property name="shoulder_lift_lower_limit" value="-6.2832" /> <!--${-pi/2}-->
+   <xacro:property name="shoulder_lift_upper_limit" value="6.2832" /> <!--0-->
    <xacro:property name="shoulder_lift_velocity_limit" value="3.1416" />
    <xacro:property name="shoulder_lift_effort_limit" value="150.0" />

Commit message: arm_ugv_edit

File: my_robot_description/src/my_robot_description/urdf/camera.xacro (robot description, xacro)
@@ -19,8 +19,11 @@
                            xyz="0 0 0" rpy="0 0 0"/>
      </link>
-     <joint name="base_camera_joint" type="fixed">
-         <parent link="base_link"/>
+     <joint name="base_camera_joint" type="revolute">
+         <parent link="hand_link"/>
          <child link="camera_link" />
-         <origin xyz="0 ${(base_width / 2.0)} ${(base_height / 2.0)+ 0.05}" rpy="0 0 ${pi/2}" />
+         <origin xyz="0 0 0.6 " rpy="0 ${pi*2} 0" />
+         <axis xyz="0 -1 0" />
+        <limit lower="0" upper="${pi*2}" effort="200" velocity="100" />
+        <dynamics friction="3.05" damping="1.0" />
      </joint>
      <!--<joint name="base_camera_joint" type="fixed">

File: my_robot_description/src/my_robot_description/urdf/common_properties.xacro (robot description, xacro)
@@ -10,4 +10,10 @@
         <color rgba="0.5 0 0 1" />
     </material>
+    <material name="orange">
+  <color rgba="1 0.5 0 1"/>
+</material>
+<material name="yellow">
+  <color rgba="1 1 0 1"/>
+</material>
     <xacro:macro name="box_inertia" params="m l w h xyz rpy">
       <inertial>

File: my_robot_description/src/my_robot_description/urdf/my_robot.urdf.xacro (robot description, xacro)
@@ -9,4 +9,18 @@
     <xacro:include filename="lidar.xacro" />
     <xacro:include filename="lidar2.xacro" />
-    <xacro:include filename="ur5.xacro" />
+    <!-- <xacro:include filename="dokari.xacro" />
+    <xacro:include filename="camera3_dokari.xacro" />
+    <xacro:include filename="camera4_dokari.xacro" />
+    <xacro:include filename="camera5_dokari.xacro" />
+    <xacro:include filename="camera6_dokari.xacro" />
+    <xacro:include filename="camera7_dokari.xacro" />
+    <xacro:include filename="camera8_dokari.xacro" /> -->
+    <!--<xacro:include filename="ur5.xacro" />-->
+    <xacro:include filename="arm.xacro" />
+    <xacro:include filename="arm_gazebo.xacro" />
+    <joint name="mobilebasearm_joint" type="fixed">
+         <parent link="base_link"/>
+         <child link="arm_base_link" />
+         <origin xyz="0.2 0 ${base_height + 0.01}" rpy="0 0 ${pi / 2.0} " />
+     </joint>
 </robot>

File: my_robot_description/src/my_robot_description/urdf/ur5.xacro (robot description, xacro)
@@ -244,5 +244,5 @@
         <parent link="lidar_link2" />
         <child link ="base_ur5" />
-        <origin xyz ="0 0 ${lidar_length2}" rpy="0 0 ${-pi}" />
+        <origin xyz ="0 0 ${lidar_length2}" rpy="0 0 ${-pi/2}" />
     </joint>
     <joint name="shoulder_pan_joint" type="revolute">
@@ -321,5 +321,5 @@
     <plugin name="gazebo_ros_joint_state_publisher"
         filename="libgazebo_ros_joint_state_publisher.so">
-       <update_rate>50</update_rate>
+       <update_rate>10</update_rate>
        <joint_name>shoulder_pan_joint</joint_name>
        <joint_name>shoulder_lift_joint</joint_name>
@@ -334,5 +334,5 @@
                 filename="libgazebo_ros_joint_pose_trajectory.so">
             <!-- Update rate in Hz -->
-            <update_rate>50</update_rate>
+            <update_rate>2</update_rate>
         </plugin>
     </gazebo>
